Commit message: new readme

File: urdf/ur5e_hand.urdf (robot description, URDF)
Before this commit: robot ur5e_hand, 24 links, 23 joints
Links:
- link base_link_inertia: geometry collision mesh filename=package://space_viz/meshes/ur5e/collision/base.stl; visual mesh filename=package://space_viz/meshes/ur5e/visual/base.dae
- link forearm_link: geometry collision mesh filename=package://space_viz/meshes/ur5e/collision/forearm.stl; visual mesh filename=package://space_viz/meshes/ur5e/visual/forearm.dae
- link hand_base: geometry collision mesh filename=package://space_viz/meshes/inspire_hand/hand_base.STL; visual mesh filename=package://space_viz/meshes/inspire_hand/hand_base.STL
- link link11: geometry collision mesh filename=package://space_viz/meshes/inspire_hand/link11.STL; visual mesh filename=package://space_viz/meshes/inspire_hand/link11.STL
- link link12: geometry collision mesh filename=package://space_viz/meshes/inspire_hand/link12.STL; visual mesh filename=package://space_viz/meshes/inspire_hand/link12.STL
- link link13: geometry collision mesh filename=package://space_viz/meshes/inspire_hand/link13.STL; visual mesh filename=package://space_viz/meshes/inspire_hand/link13.STL
- link link14: geometry collision mesh filename=package://space_viz/meshes/inspire_hand/link14.STL; visual mesh filename=package://space_viz/meshes/inspire_hand/link14.STL
- link link21: geometry collision mesh filename=package://space_viz/meshes/inspire_hand/link21.STL; visual mesh filename=package://space_viz/meshes/inspire_hand/link21.STL
- link link22: geometry collision mesh filename=package://space_viz/meshes/inspire_hand/link22.STL; visual mesh filename=package://space_viz/meshes/inspire_hand/link22.STL
- link link31: geometry collision mesh filename=package://space_viz/meshes/inspire_hand/link31.STL; visual mesh filename=package://space_viz/meshes/inspire_hand/link31.STL
- link link32: geometry collision mesh filename=package://space_viz/meshes/inspire_hand/link32.STL; visual mesh filename=package://space_viz/meshes/inspire_hand/link32.STL
- link link41: geometry collision mesh filename=package://space_viz/meshes/inspire_hand/link41.STL; visual mesh filename=package://space_viz/meshes/inspire_hand/link41.STL
- link link42: geometry collision mesh filename=package://space_viz/meshes/inspire_hand/link42.STL; visual mesh filename=package://space_viz/meshes/inspire_hand/link42.STL
- link link51: geometry collision mesh filename=package://space_viz/meshes/inspire_hand/link51.STL; visual mesh filename=package://space_viz/meshes/inspire_hand/link51.STL
- link link52: geometry collision mesh filename=package://space_viz/meshes/inspire_hand/link52.STL; visual mesh filename=package://space_viz/meshes/inspire_hand/link52.STL
- link shoulder_link: geometry collision mesh filename=package://space_viz/meshes/ur5e/collision/shoulder.stl; visual mesh filename=package://space_viz/meshes/ur5e/visual/shoulder.dae
- link upper_arm_link: geometry collision mesh filename=package://space_viz/meshes/ur5e/collision/upperarm.stl; visual mesh filename=package://space_viz/meshes/ur5e/visual/upperarm.dae
- link wrist_1_link: geometry collision mesh filename=package://space_viz/meshes/ur5e/collision/wrist1.stl; visual mesh filename=package://space_viz/meshes/ur5e/visual/wrist1.dae
- link wrist_2_link: geometry collision mesh filename=package://space_viz/meshes/ur5e/collision/wrist2.stl; visual mesh filename=package://space_viz/meshes/ur5e/visual/wrist2.dae
- link wrist_3_link: geometry collision mesh filename=package://space_viz/meshes/ur5e/collision/wrist3.stl; visual mesh filename=package://space_viz/meshes/ur5e/visual/wrist3.dae
